Commit message: some changes

File: description/urdf/PanTiltMerge.xacro (robot description, xacro)
@@ -4,4 +4,9 @@
 <xacro:include filename="$(find pioneer_playground)/description/urdf/PanTiltMerge.trans" />
 <xacro:include filename="$(find pioneer_playground)/description/urdf/PanTiltMerge.gazebo" />
+  <link name="world"/>
+  <joint name="fixed" type="fixed">
+    <parent link="world"/>
+    <child link="base_link"/>
+  </joint>
 <link name="base_link">
   <inertial>
